Commit message: i

File: src/allegro_hand_description/allegro_hand_description_right.xacro (robot description, xacro)
@@ -119,5 +119,5 @@
                     <color rgba=".2 .2 .2 1"/>
                 </material>
-                <origin rpy="${180*DEG2RAD} 0 0" xyz="0 0 0"/>
+                <origin rpy="${DEG2RAD} 0 0" xyz="0 0 0"/>
             </visual>
             <collision>
